File: fonte.sch (EAGLE design)
At the start: 52 parts, among them IC1 LM358D, IC2 REG1117F, IC3 7812DT, IC5 PIC16F877PT, Q2 BSA223SP, Q5 2N2907

Commit message: teste de atualização.
testando a alteração do meu arquivo, não entendo nada de github ainda...
Connections:
- removed net N$3: IC3.VI
- net 30V: now also IC3.VI
Other:
- note added: "Borne de saida já estabilizado"
- note added: "Borne para receber a corrente vinda dos capacitores e retificadores"
- note added: "Proteção de sobretensão, caso alguma coisa de errado antes do FET, ele pode cortar a alimentação da parte logica da fonte"
- moved on the sheet: 10K, 10K1, 10K2, 1K, IC1A, IC2, IC3, Q2, UART, ZD1

Commit message: identificações das ligações
melhorei a identificação das partes
Parts:
- removed 10K10: 2k, adafruit:R-US_R0603
- removed 10K9: 10k, adafruit:R-US_R0603
- removed ESTABILIZADO: (no value), con-ptr500:AK300/2
- removed R12: 5k6, adafruit:R-US_R0603
- added C6: 100K, adafruit:C-USC1812
- added R-SHUNT: 25R, adafruit:R-US_R0603
- added R24: 2k, adafruit:R-US_R0603
- added R25: 10k, adafruit:R-US_R0603
- added SAIDA: (no value), con-ptr500:AK300/2
- added T1: 2N3055, transistor:2N3055
- S1: value RACON12 -> reset
- renumbered 10K to R20, 10K1 to R21, 10K2 to R23, 10K3 to R26, 10K4 to R15, 10K5 to R16, 10K6 to R17, 10K7 to R19, 10K8 to R18, 1K to R22
Connections:
- removed net +B: ESTABILIZADO-1.KL
- removed net 3V: ICSP.2
- removed net AJUSTE-CORRENTE: C1.+, R7.2
- removed net AJUSTE-TENSAO: C2.+, R9.2
- removed net N$20: D2.C, Q5.B, R13.2
- new net AJUSTE-TENSAO-E-CORRENTE: C1.+, C2.+, D2.C, Q5.B, R13.2, R7.2, R9.2
- new net N$3: SAIDA-1.KL, T1.E
- net 30V: now also C6.1, T1.C
- net 5V: now also ICSP.2
- net DIREITA: no longer IC5.INT/RB0
- net GND: now also R-SHUNT.2, R24.1; no longer 10K10.1, R12.2
- net N$23: now also C6.2, T1.B
- net N$8: now also R25.1; no longer 10K9.1
- net SHUNT: now also R-SHUNT.1, SAIDA-2.KL; no longer ESTABILIZADO-2.KL, R12.1
- net SONDA-TENSAO: now also R24.2, R25.2; no longer 10K10.2, 10K9.2
Other:
- note removed: "Borne de saida já estabilizado"
- moved on the sheet: C1, C2, R11, R2, R3, R6, R7, R8, R9, S1, SONDA-SAIDA
