File: fonte.sch (EAGLE design)
At the start: 54 parts, among them IC1 LM358D, IC2 REG1117F, IC3 7812DT, IC5 PIC16F877PT, Q2 BSA223SP, Q5 2N2907, T1 2N3055

Commit message: divulgando.
Other:
- note added: "1 - Alimentação do NTC 2 - Retorno do NTC 3 - +12v alimentação do ventilador 4 - GND para o ventilador Label cooler - Sinal para acionar o cooler."
- note added: "Não é pra ser o 2n3055, mas como eu não encontro o package do 2sc5200, vou deixar esse transistor mesmo por enquanto."
Changed lines of the file:
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@@
  errado antes do FET, ele pode cortar a
  alimentação da parte logica da fonte</text>
+<text x="71.12" y="147.32" size="1.4224" layer="97" ratio="3">1 - Alimentação do NTC
+2 - Retorno do NTC
+3 - +12v alimentação do ventilador
+4 - GND para o ventilador
+Label cooler - Sinal para acionar o cooler.</text>
+<text x="109.22" y="81.28" size="1.4224" layer="97" ratio="3">Não é pra ser o 2n3055, mas como
+ eu não encontro o package do
+2sc5200, vou deixar esse transistor
+ mesmo por enquanto.</text>
 </plain>
 <instances>
